File: BURC_For_All_Transmitters/Angle&Ana&Sw/Angle&Ana&Sw.kicad_pcb (KiCad board)
At the start: 2 copper layers, 85.1 x 38.7 mm, 23 parts, among them J1 Conn_01x04, J10 Conn_ButtonsRight, J10B1 Conn_ButtonsRight, J2 I2C_INPUT, J3 I2C_INPUT, J4 I2C_INPUT, J5 I2C_INPUT, J6 Conn_ToButtonsLeft, J7 Conn_FromButtonsLeft, J9 Conn_ButtonsLeft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

Commit message: Swap CPPM_IN/CPPM_OUT
Connections:
- J1 pad 1: /CPPM_IN -> /CPPM_OUT
- J1 pad 2: /CPPM_OUT -> /CPPM_IN
- U3 pad D8: /CPPM_OUT -> /CPPM_IN
- U3 pad D9: /CPPM_IN -> /CPPM_OUT
Routing:
- net /CPPM_OUT: track 23.0 -> 26.0 mm
- net /CPPM_IN: track 26.0 -> 23.0 mm
Other:
- board text added: "CPPM_OUT/SBUS_OUT"
- board text removed: "CPPM/SBUS_OUT"
