File: BURC_For_All_Transmitters/MultiSwitch_Mcp23017_MiniSwitch/MultiSwitch_Mcp23017_MiniSwitch.kicad_pcb (KiCad board)
At the start: 2 copper layers, 85.1 x 38.7 mm, 27 parts, among them J1 MPC23017_MODULE, J2 I2C_INPUT, J3 I2C_INPUT, J4 I2C_INPUT, J5 I2C_INPUT, J6 PCF8574, J7 PCF8574, J8 PCF8575, SW1 SW_SPST, SW10 SW_SPST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

Commit message: Update drill switch
Routing:
- net GND: track 30.0 -> 32.1 mm
- net /C6: track 21.8 -> 22.6 mm
- net /C2: track 30.0 -> 30.6 mm
- net /C3: track 25.2 -> 25.8 mm
- net /C13: track 16.3 -> 16.8 mm
- net /SCL: track 151.1 -> 151.6 mm
